File: Hardwares/Elecraft_K1_Remake.kicad_sch (KiCad schematic)
At the start: 122 parts, among them J1 RF_IN, J10 Conn_01x01, J11 Conn_01x01, J12 Conn_01x01, J13 Conn_01x01, J14 Conn_01x01, J2 PWR_12V, J3 Premix_Filter, J4 Freq_Counter, J5 VFO_Out, J6 Outer_Ctrl, J7 SMTR, J8 Audio, J9 Conn_01x01, Q1 S9018, Q2 2N3904, Q3 2N3906, Q4 2N3904, Q5 2N7000, Q6 2N3906, Q7 MPSA14_EBC, Q8 2N7000, T1 4:20, T2 5:20, U1 L78L05_TO92, U2 SA602, U3 L78L05_TO92, U4 SA602, U5 LM386, U6 SA602, U7 LM380N-8, Y1 4.915MHz, Y2 4.915MHz, Y3 4.915MHz, Y4 4.915MHz, Y5 4.915MHz

Commit message: Add files via upload
Parts:
- removed C28: 1u, Capacitor_THT:C_Disc_D5.1mm_W3.2mm_P5.00mm, symbol Device:C
- removed C29, C30, C42: 10u, Capacitor_THT:CP_Radial_D5.0mm_P2.50mm, symbol Device:C_Polarized
- removed C31, C40: .01u, Capacitor_THT:C_Disc_D5.1mm_W3.2mm_P5.00mm, symbol Device:C
- removed C38, C39: .1u, Capacitor_THT:C_Disc_D5.1mm_W3.2mm_P5.00mm, symbol Device:C
- removed C41: 2.2u, Capacitor_THT:CP_Radial_D5.0mm_P2.50mm, symbol Device:C_Polarized
- removed C44: 220, Capacitor_THT:C_Disc_D5.1mm_W3.2mm_P5.00mm, symbol Device:C
- removed D6: 1N5711, Diode_THT:D_DO-35_SOD27_P7.62mm_Horizontal, symbol Diode:1N5711
- removed J7: SMTR, Connector_JST:JST_XH_S2B-XH-A_1x02_P2.50mm_Horizontal, symbol Connector_Generic:Conn_01x02
- removed JP1: JMP, Connector_Wire:SolderWire-0.5sqmm_1x02_P4.6mm_D0.9mm_OD2.1mm, symbol Jumper:Jumper_2_Bridged
- removed Q5, Q8: 2N7000, Package_TO_SOT_THT:TO-92_Inline, symbol Transistor_FET:2N7000
- removed Q6: 2N3906, Package_TO_SOT_THT:TO-92_Inline, symbol Transistor_BJT:2N3906
- removed Q7: MPSA14_EBC, Package_TO_SOT_THT:TO-92_Inline, symbol Device:Q_NPN_Darlington_EBC
- removed R17: 2.7k, Resistor_THT:R_Axial_DIN0207_L6.3mm_D2.5mm_P7.62mm_Horizontal, symbol Device:R
- removed R18: 2.2M, Resistor_THT:R_Axial_DIN0207_L6.3mm_D2.5mm_P7.62mm_Horizontal, symbol Device:R
- removed R19: 47k, Resistor_THT:R_Axial_DIN0207_L6.3mm_D2.5mm_P7.62mm_Horizontal, symbol Device:R
- removed R26: 27k, Resistor_THT:R_Axial_DIN0207_L6.3mm_D2.5mm_P7.62mm_Horizontal, symbol Device:R
- removed RV3: 50k, Potentiometer_THT:Potentiometer_Piher_PT-6-V_Vertical, symbol Device:R_Potentiometer
- removed U5: LM386, Package_DIP:DIP-8_W7.62mm_Socket, symbol Amplifier_Audio:LM386
- added C13: 22u, Capacitor_THT:CP_Radial_D8.0mm_P2.50mm, symbol Device:C_Polarized
- added C32, C34, C36: .01u, Capacitor_THT:C_Disc_D5.1mm_W3.2mm_P5.00mm, symbol Device:C
- added C35: 180, Capacitor_THT:C_Disc_D5.1mm_W3.2mm_P5.00mm, symbol Device:C
- added D6: 1N4148, Diode_THT:D_DO-35_SOD27_P7.62mm_Horizontal, symbol Diode:1N4148
- added D7: ISV149, Package_TO_SOT_THT:TO-92-2, symbol Device:D_Capacitance
- added J14: IF_Out, Connector_JST:JST_XH_S2B-XH-A_1x02_P2.50mm_Horizontal, symbol Connector_Generic:Conn_01x02
- added L2: 4.7u, Inductor_THT:L_Axial_L7.0mm_D3.3mm_P12.70mm_Horizontal_Fastron_MICC, symbol Device:L
- added Q1: 2N7000, Package_TO_SOT_THT:TO-92_Inline, symbol Transistor_FET:2N7000
- added Q6: 2N3904, Package_TO_SOT_THT:TO-92_Inline, symbol Transistor_BJT:2N3904
- added R6: 1k, Resistor_THT:R_Axial_DIN0207_L6.3mm_D2.5mm_P7.62mm_Horizontal, symbol Device:R
- added U6: MC1350, Package_DIP:DIP-8_W7.62mm_Socket, symbol 0_Self_Defined_Symbol:MC1350
- added Y5, Y6: 4.915MHz, Crystal:Crystal_HC49-U_Vertical, symbol Device:Crystal
- C16: renamed from C11; value .001u -> 1000
- C17: renamed from C12; value .001u -> 1000
- C33: value .01u -> 0.47u
- C37: value .01u -> 100
- J9: renamed from J5; value VFO_Out -> PreMix_Out
- L1: value 4.4u -> 47u
- L3: renamed from L2; value 33u -> 47u
- R20: value 47k -> 5k
- R21: value 47k -> 5.6k
- R22: value 1.8k -> 3.9k
- R23: value 47k -> 100k
- renumbered C24 to C1, C6 to C10, C7 to C11, C8 to C12, C9 to C14, C10 to C15, C47 to C18, C13 to C19, C25 to C2, C45 to C20, C46 to C21, C14 to C22, C15 to C23, C17 to C24, C18 to C25, C16 to C26, C20 to C27, C19 to C28, C22 to C29, C26 to C3, C23 to C30, C21 to C31, C27 to C38, C32 to C39, C1 to C4, C34 to C40, C35 to C41, C36 to C42, C2 to C5, C3 to C6, C4 to C7, C5 to C8, C43 to C9, J4 to J10, J12 to J11, J13 to J12, J14 to J13, J8 to J3, J6 to J4, J3 to J5, J9 to J6, J10 to J7, J11 to J8, Q1 to Q2, Q2 to Q3, Q3 to Q4, Q4 to Q5, R16 to R1, R7 to R10, R25 to R11, R8 to R12, R9 to R13, R10 to R14, R13 to R15, R11 to R16, R14 to R17, R12 to R18, R15 to R19, R1 to R2, R2 to R3, R3 to R4, R4 to R5, R5 to R7, R24 to R8, R6 to R9, RV4 to RV2, RV2 to RV3, U7 to U3, U3 to U4, U4 to U5, U6 to U7, Y5 to Y7
Connections:
- net +12V: now also C33.2, R21.1, L2.2, U6.1 (OUTA), U6.2 (VCC)
- net 6R/AUX: now also Q3.3 (C)
- net GND: now also C33.1, C32.2, C35.1, C36.2, D7.2 (A), J14.2 (Pin_2), Q6.1 (E), R6.2, U6.3 (GND), U6.7 (GND); no longer C37.2, C9.2, RV2.3, U3.2 (+)
- net at C1.1, R1.1: now also Q1.2 (G)
- net at C37.1: now also Q6.3 (C); no longer D5.2 (A)
- net at R20.2: now also U6.5 (AGC)
- net at U3.8 (BYPASS): now also C13.1
- net at C3.2: now also RV2.3, Q1.1 (S)
- net at C2.2: now also C9.1, RV2.1, U3.2 (+), Q1.3 (D)
- net BW_Ctrl: now reaches R23.2
- net BW_Ctrl: now also C29.1, R15.2, R17.2, R19.2, RV3.2
- net Coil_2A: now reaches C30.2, T2.2 (AB)
- net Coil_2A: now also R22.1
- net at U7.1 (IN_A): now also Y6.2; no longer T2.4 (SB)
- net 6R/AUX1: no longer names the net of D5.1 (K)
- net 6R/AUX1: now also T2.3 (SA), C32.1, D6.2 (A), U6.6 (INB); no longer Q3.3 (C)
- net Coil_1: no longer names the net of C6.1, T1.3 (SA), U2.2 (IN_B)
- net Coil_1: no longer R22.1
- net Coil_2: no longer names the net of C38.1, U7.2 (IN_B)
- net Coil_2: no longer R22.2, T2.3 (SA)
- net XFIL/TONE renamed SideTone
- net SideTone: now also C13.2, R6.1
- net ~{AGC OFF} renamed AGC
- net AGC: now also R20.1
- new net: D7.1 (K), R23.1, Y5.2, Y6.1
- new net: C34.1, J14.1 (Pin_1)
- new net: C34.2, C35.2, C37.2, L2.1, R21.2, U6.8 (OUTB), Y5.1
- new net: D5.2 (A), D6.1 (K), T2.4 (SB), U6.4 (INA)
- new net: C9.2, RV2.2, U3.3 (-)
- new net: C36.1, Q6.2 (B), R22.2
Other:
- note added: "1st Internal Freq Filter"
- note added: "2nd IF Filter"
- note added: "IF Amp"
- note removed: "AF PreAmp"
- note removed: "AGC"
- note removed: "AGC Adjustment"
- note removed: "For routing only"
- note removed: "Internal Freq Filter"
- moved on the sheet: C1, C10, C11, C12, C14, C15, C16, C17, C18, C19, C2, C20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
